Commit message: SCM working locomotion policy, Refresh docs

File: models/go1/go1_chrono.urdf (robot description, URDF)
Before this commit: robot go1, 38 links, 37 joints
Links:
- link FL_calf: geometry collision box size=0.193 0.016 0.016; visual mesh filename=meshes/calf.dae scale=1 1 1
- link FR_calf: geometry collision box size=0.193 0.016 0.016; visual mesh filename=meshes/calf.dae scale=1 1 1
- link RL_calf: geometry collision box size=0.193 0.016 0.016; visual mesh filename=meshes/calf.dae scale=1 1 1
- link RR_calf: geometry collision box size=0.193 0.016 0.016; visual mesh filename=meshes/calf.dae scale=1 1 1
